File: hardware/KiCad/Sequencer Pi Pico 4 layers V3.kicad_pcb (KiCad board)
At the start: 4 copper layers, 55 x 100 mm, 146 parts, among them J1 SMA, J10 Screw_Terminal, J11 Screw_Terminal, J12 Screw_Terminal, J2 SMA, J3 SMA, J4 SMA, J5 Screw_Terminal, J6 Screw_Terminal, J7 Screw_Terminal, J8 Screw_Terminal, J9 Screw_Terminal, P1 1K, Q1 MMBF170, Q10 MMBF170, Q11 IRF9Z24S, Q12 MMBF170, Q13 MMBTA13, Q14 IRF9Z24S, Q15 MMBTA13, Q16 MMBF170, Q2 MMBF170, Q3 MMBF170, Q4 MMBF170, Q5 IRF9Z24S, Q6 MMBTA13, Q7 MMBF170, Q8 IRF9Z24S, Q9 MMBF170, U1 MAR-6, U2 LM7805_TO220

Commit message: Fixed circuit for latched relays
Parts:
- added D29: BAV16W, Diode_SMD:D_SOD-323_HandSoldering, B.Cu at (146.9, 128.1)
- added D30: BAV16W, Diode_SMD:D_SOD-323_HandSoldering, B.Cu at (146.9, 125.6)
- R35: value 10K -> 3K3
- R8: value VPR220 50 / * -> VPR220 50
- moved R31 0.80 mm to (147.1, 130.3)
Connections:
- net /MCU Logic/TR_RELAY_FB renamed /MCU Logic/RELAY_FB
- R38 pad 2: /MCU Logic/TR_RELAY_TX -> Net-(D29-K)
- R44 pad 2: /MCU Logic/TR_RELAY_RX -> Net-(D30-K)
Routing:
- net Net-(D30-K): track 0.00 -> 13.2 mm, vias 0 -> 2
- net /MCU Logic/TR_RELAY_RX: track 35.4 -> 24.8 mm, vias 3 -> 2
- net /MCU Logic/TR_RELAY_TX: track 25.1 -> 15.0 mm, vias 2 -> 0
- net Net-(D29-K): track 0.00 -> 7.69 mm, vias 0 -> 2
Other:
- board text added: "260423"
- board text removed: "260326"
